Commit message: V48-C: add realistic mass (servo/SBC/battery) to base_link
base_link mass: 2.80 → 4.04 kg (+1.24kg)
Added: 12 servos (0.66), SBC (0.05), battery (0.30), wiring (0.20), PCA9685 (0.03)
Inertia scaled proportionally (×1.443)

force_usd_conversion=True for URDF mass change to take effect.

Heavier body = more stable standing, more realistic dynamics,
better sim-to-real transfer potential.

File: assets/robots/spot_micro/spotmicroai_realistic_inertia.urdf (robot description, URDF)
Before this commit: robot SpotMicroAI, 25 links, 24 joints
Links:
- link base_link: mass 2.80 -> 4.04

Commit message: V48-D: realistic mass distribution + MG996R torque limit
Mass distributed to joints (not all on base):
- base_link: 2.80 → 3.60 (+0.80: battery/SBC/PCA/wiring/body servos)
- leg_link ×4: 0.15 → 0.205 (+0.055: 1 servo each)
- foot_link ×4: 0.10 → 0.155 (+0.055: 1 servo each)
- Total added: 0.80 + 0.22 + 0.22 = 1.24kg

Torque realistic to MG996R servo:
- saturation_effort: 15.0 → 1.5 N·m (MG996R stall=1.08, +40% margin)
- effort_limit: 15.0 → 1.5 N·m
- stiffness=15 maintained (saturates at >0.1rad error = realistic)

File: assets/robots/spot_micro/spotmicroai_realistic_inertia.urdf (robot description, URDF)
Before this commit: robot SpotMicroAI, 25 links, 24 joints
Links:
- link base_link: mass 4.04 -> 3.60
- link front_left_foot_link: mass 0.1 -> 0.155
- link front_left_leg_link: mass 0.15 -> 0.205
- link front_right_foot_link: mass 0.1 -> 0.155
- link front_right_leg_link: mass 0.15 -> 0.205
- link rear_left_foot_link: mass 0.1 -> 0.155
- link rear_left_leg_link: mass 0.15 -> 0.205
- link rear_right_foot_link: mass 0.1 -> 0.155
- link rear_right_leg_link: mass 0.15 -> 0.205

Commit message: V49: restore V48-B baseline (original mass + effort=15 + leg=-0.97)
Reverted V48-C/D realism changes that broke walking baseline:
- URDF mass: restored to original 5.3kg (was 6.54kg)
- effort: restored to 15.0 N·m (was 1.5/5.0)
- Standing pose leg=-0.97 kept (verified improvement)

Two-track strategy:
1. Walking baseline track: V49 (get walking right first)
2. Realism track: separate future versions (mass/torque sim-to-real)

File: assets/robots/spot_micro/spotmicroai_realistic_inertia.urdf (robot description, URDF)
Before this commit: robot SpotMicroAI, 25 links, 24 joints
Links:
- link base_link: mass 3.60 -> 2.80
- link front_left_foot_link: mass 0.155 -> 0.1
- link front_left_leg_link: mass 0.205 -> 0.15
- link front_right_foot_link: mass 0.155 -> 0.1
- link front_right_leg_link: mass 0.205 -> 0.15
- link rear_left_foot_link: mass 0.155 -> 0.1
- link rear_left_leg_link: mass 0.205 -> 0.15
- link rear_right_foot_link: mass 0.155 -> 0.1
- link rear_right_leg_link: mass 0.205 -> 0.15

Commit message: V57.B1: zero-action standing 달성 — ImplicitActuator 전환 + 물리 디버깅
3대 근본 원인 발견 및 해결:
1. init_z에 toe sphere radius(0.02m) 미포함 → 20mm 지면 관통 → impulse
2. URDF velocity=10 = DCMotor velocity_limit=10 → bang-bang 진동
3. DCMotor velocity-dependent saturation → crouched equilibrium 수렴

해결: ImplicitActuatorCfg 전환 (PhysX 연속시간 PD, velocity saturation 제거)
- effort_limit=15 유지 (토크 제한 현실성 보존)
- 관절별 차등 gain: shoulder=12/4, leg=28/5, foot=8/2
- URDF velocity 10→20, max_depenetration 1.0→0.2
- init_z=0.185 (loaded equilibrium 근처)
- target_height 0.22→0.18 (loaded eq 기반)

결과: height=0.1441에서 300+ steps 완벽 정지 (소수점 4자리 고정)

File: assets/robots/spot_micro/spotmicroai_realistic_inertia.urdf (robot description, URDF)
Before this commit: robot SpotMicroAI, 25 links, 24 joints
Joints:
- joint front_left_foot: limit lower=-0.1 upper=2.59 effort=1000.0 velocity=10.0 -> lower=-0.1 upper=2.59 effort=1000.0 velocity=20.0
- joint front_left_leg: limit lower=-2.666 upper=1.548 effort=1000.0 velocity=10.0 -> lower=-2.666 upper=1.548 effort=1000.0 velocity=20.0
- joint front_left_shoulder: limit lower=-0.548 upper=0.548 effort=1000.0 velocity=10.0 -> lower=-0.548 upper=0.548 effort=1000.0 velocity=20.0
- joint front_right_foot: limit lower=-0.1 upper=2.59 effort=1000.0 velocity=10.0 -> lower=-0.1 upper=2.59 effort=1000.0 velocity=20.0
- joint front_right_leg: limit lower=-2.666 upper=1.548 effort=1000.0 velocity=10.0 -> lower=-2.666 upper=1.548 effort=1000.0 velocity=20.0
- joint front_right_shoulder: limit lower=-0.548 upper=0.548 effort=1000.0 velocity=10.0 -> lower=-0.548 upper=0.548 effort=1000.0 velocity=20.0
- joint rear_left_foot: limit lower=-0.1 upper=2.59 effort=1000.0 velocity=10.0 -> lower=-0.1 upper=2.59 effort=1000.0 velocity=20.0
- joint rear_left_leg: limit lower=-2.666 upper=1.548 effort=1000.0 velocity=10.0 -> lower=-2.666 upper=1.548 effort=1000.0 velocity=20.0
- joint rear_left_shoulder: limit lower=-0.548 upper=0.548 effort=1000.0 velocity=10.0 -> lower=-0.548 upper=0.548 effort=1000.0 velocity=20.0
- joint rear_right_foot: limit lower=-0.1 upper=2.59 effort=1000.0 velocity=10.0 -> lower=-0.1 upper=2.59 effort=1000.0 velocity=20.0
- joint rear_right_leg: limit lower=-2.666 upper=1.548 effort=1000.0 velocity=10.0 -> lower=-2.666 upper=1.548 effort=1000.0 velocity=20.0
- joint rear_right_shoulder: limit lower=-0.548 upper=0.548 effort=1000.0 velocity=10.0 -> lower=-0.548 upper=0.548 effort=1000.0 velocity=20.0

Commit message: V59: DCMotor(STS3215 3Nm) + URDF mass 실물 기준 수정 (5.3kg→1.41kg)
- URDF 전체 질량 실물 BOM 기반 재설정 (base 0.50, lidar 0.17 등)
- base 루트 링크 inertial 누락 발견 → PhysX 1kg 기본값 문제 해결
- DCMotor: effort=3Nm, stiffness=5, damping=0.5 (STS3215 실제 스펙)
- 대칭 Z-bend init pose (leg=-0.52, foot=1.04, shoulder=±0.05)
- Stand test 검증: h=149mm, pitch=-3°, 500 step 안정
- URDF velocity 20→100 (PhysX가 DCMotor를 간섭하지 않도록)
- V59 stand-first env 블록 추가
- flat_orientation_bonus reward 추가
- stance search 유틸리티 스크립트 추가

File: assets/robots/spot_micro/spotmicroai_realistic_inertia.urdf (robot description, URDF)
Before this commit: robot SpotMicroAI, 25 links, 24 joints
Links:
- link base: mass None -> 0.001
- link base_link: mass 2.80 -> 0.50
- link front_left_foot_link: mass 0.1 -> 0.04
- link front_left_leg_link: mass 0.15 -> 0.04
- link front_left_shoulder_link: mass 0.10 -> 0.065
- link front_left_toe_link: mass 0.05 -> 0.01
- link front_link: mass 0.20 -> 0.06
- link front_right_foot_link: mass 0.1 -> 0.04
- link front_right_leg_link: mass 0.15 -> 0.04
- link front_right_shoulder_link: mass 0.10 -> 0.065
- link front_right_toe_link: mass 0.05 -> 0.01
- link lidar_link: mass 0.50 -> 0.17
- link rear_left_foot_link: mass 0.1 -> 0.04
- link rear_left_leg_link: mass 0.15 -> 0.04
- link rear_left_shoulder_link: mass 0.10 -> 0.065
- link rear_left_toe_link: mass 0.05 -> 0.01
- link rear_link: mass 0.20 -> 0.06
- link rear_right_foot_link: mass 0.1 -> 0.04
- link rear_right_leg_link: mass 0.15 -> 0.04
- link rear_right_shoulder_link: mass 0.10 -> 0.065
- link rear_right_toe_link: mass 0.05 -> 0.01
Joints:
- joint front_left_foot: limit lower=-0.1 upper=2.59 effort=1000.0 velocity=20.0 -> lower=-0.1 upper=2.59 effort=1000.0 velocity=100.0
- joint front_left_leg: limit lower=-2.666 upper=1.548 effort=1000.0 velocity=20.0 -> lower=-2.666 upper=1.548 effort=1000.0 velocity=100.0
- joint front_left_shoulder: limit lower=-0.548 upper=0.548 effort=1000.0 velocity=20.0 -> lower=-0.548 upper=0.548 effort=1000.0 velocity=100.0
- joint front_right_foot: limit lower=-0.1 upper=2.59 effort=1000.0 velocity=20.0 -> lower=-0.1 upper=2.59 effort=1000.0 velocity=100.0
- joint front_right_leg: limit lower=-2.666 upper=1.548 effort=1000.0 velocity=20.0 -> lower=-2.666 upper=1.548 effort=1000.0 velocity=100.0
- joint front_right_shoulder: limit lower=-0.548 upper=0.548 effort=1000.0 velocity=20.0 -> lower=-0.548 upper=0.548 effort=1000.0 velocity=100.0
- joint rear_left_foot: limit lower=-0.1 upper=2.59 effort=1000.0 velocity=20.0 -> lower=-0.1 upper=2.59 effort=1000.0 velocity=100.0
- joint rear_left_leg: limit lower=-2.666 upper=1.548 effort=1000.0 velocity=20.0 -> lower=-2.666 upper=1.548 effort=1000.0 velocity=100.0
- joint rear_left_shoulder: limit lower=-0.548 upper=0.548 effort=1000.0 velocity=20.0 -> lower=-0.548 upper=0.548 effort=1000.0 velocity=100.0
- joint rear_right_foot: limit lower=-0.1 upper=2.59 effort=1000.0 velocity=20.0 -> lower=-0.1 upper=2.59 effort=1000.0 velocity=100.0
- joint rear_right_leg: limit lower=-2.666 upper=1.548 effort=1000.0 velocity=20.0 -> lower=-2.666 upper=1.548 effort=1000.0 velocity=100.0
- joint rear_right_shoulder: limit lower=-0.548 upper=0.548 effort=1000.0 velocity=20.0 -> lower=-0.548 upper=0.548 effort=1000.0 velocity=100.0
